Commit message: 11-30-2024 Build
Bugfixing & adjusting dependencies.

File: autonomy/snow_white_description/install/snow_white_description/share/snow_white_description/src/description/snow_white_description_v2.urdf (robot description, URDF)
Before this commit: robot snow_white_v2, 22 links, 21 joints
Joints:
- joint left_augur_wheel_joint: type continuous -> fixed
- joint right_augur_wheel_joint: type continuous -> fixed

File: autonomy/snow_white_description/install/snow_white_description/share/snow_white_description/src/description/snow_white_description_v2_backup.urdf (robot description, URDF)
Before this commit: robot snow_white_v2, 22 links, 21 joints
Joints:
- joint left_augur_wheel_joint: type continuous -> fixed
- joint right_augur_wheel_joint: type continuous -> fixed
